Commit message: zamieniono teleport na plyniecie z dana predkoscia; wyrzucono parametry nodow do configow

File: src/xm540_bringup/urdf/xm540_manipulator_isaac.urdf (robot description, URDF)
Before this commit: robot xm540_manipulator, 5 links, 4 joints
Links:
- added link boat_x_link, mass 0.001
- added link boat_y_link, mass 0.001
- added link world, mass 0.001
Joints:
- added joint boat_to_base: type fixed, parent boat_y_link, child base_link, origin xyz=0 0 0 rpy=3.14159 0 0
- added joint joint_boat_x: type prismatic, parent world, child boat_x_link, origin xyz=0 0 0 rpy=0 0 0, axis 1 0 0, limit lower=-2000 upper=2000 effort=100000 velocity=100
- added joint joint_boat_y: type prismatic, parent boat_x_link, child boat_y_link, origin xyz=0 0 0 rpy=0 0 0, axis 0 1 0, limit lower=-2000 upper=2000 effort=100000 velocity=100

Commit message: wprowadzenie zmiennej w configu symulacji okreslajacej skale swiata; zmieniono jej odmyslan wartosc z x10 na x1; nowe waypointy pod nowa skale; dodano liczenie czasu trwania scenariusza; dodano opcje by waypoint generator dostosowal siatke pod czas trwania misji; usunieto kolizje manipulatora z jeziorem

File: src/xm540_bringup/urdf/xm540_manipulator_isaac.urdf (robot description, URDF)
Before this commit: robot xm540_manipulator, 8 links, 7 joints
Links:
- link link_0: geometry visual mesh filename=package://xm540_bringup/meshes/link_0.stl scale=0.001 0.001 0.001
- link link_1: geometry visual mesh filename=package://xm540_bringup/meshes/link_1.stl scale=0.001 0.001 0.001
- link link_2: geometry visual mesh filename=package://xm540_bringup/meshes/link_2.stl scale=0.001 0.001 0.001
